Commit message: fixed gazebo simulation

File: urdf/simplebot.urdf.xacro (robot description, xacro)
@@ -7,5 +7,4 @@
   <xacro:property name="M_PI" value="3.1415926535897931" />
   <xacro:property name="wheel_width" value="0.01" />
-  <!-- This is the wheel radius for the robot height, the one for the odometry is in volksbot_node.cpp  -->
   <xacro:property name="wheel_radius" value="0.0245" />
   <xacro:property name="axis_length" value="0.160" />
@@ -42,5 +41,5 @@
     </inertial>
   </link>
-  <xacro:macro name="volksbot_wheel" params="name xyz rotate_visual friction">
+  <xacro:macro name="wheel" params="name xyz rotate_visual friction">
     <link name="${name}_wheel_link">
       <visual>
@@ -56,6 +55,14 @@
         <origin xyz="0 0 0" rpy="${M_PI/2} 0 0" />
         <geometry>
-          <mesh filename="package://simplebot_driver/model/simplebot_wheel.stl"/>
+            <cylinder length="${wheel_width}" radius="${wheel_radius}"/>
         </geometry>
+        <surface>
+          <friction>
+            <ode>
+              <mu>0.1</mu>
+              <mu2>0.1</mu2>
+            </ode>
+          </friction>
+        </surface>
       </collision>
       <inertial>
@@ -73,16 +80,25 @@
       <axis xyz="0 1 0"/>
     </joint>
+    <gazebo reference="${name}_wheel_link">
+      <mu1>1.0</mu1>
+      <mu2>1.0</mu2>
+      <material>Gazebo/Black</material>
+      <kp>100000.0</kp>
+      <kd>10.0</kd>
+      <fdir1>1 0 0</fdir1>
+      <maxVel>1.0</maxVel>
+      <minDepth>0.00</minDepth>
+      <selfCollide>false</selfCollide>
+    </gazebo>
   </xacro:macro>
-  <xacro:volksbot_wheel name="left_front" xyz="${wheel_x_offset} ${axis_length/2} ${wheel_z_offset}" rotate_visual="1" friction="1.0" />
-  <xacro:volksbot_wheel name="left_rear" xyz="${-wheel_x_offset} ${axis_length/2} ${wheel_z_offset}" rotate_visual="1" friction="1.0" />
-  <xacro:volksbot_wheel name="right_front" xyz="${wheel_x_offset} ${-axis_length/2} ${wheel_z_offset}" rotate_visual="0" friction="1.0" />
-  <xacro:volksbot_wheel name="right_rear" xyz="${-wheel_x_offset} ${-axis_length/2} ${wheel_z_offset}" rotate_visual="0" friction="1.0" />
-  <!-- base_footprint is a fictitious link(frame) that is on the ground right below base_link origin,
-       navigation stack depends on this frame -->
+  <xacro:wheel name="left_front" xyz="${wheel_x_offset} ${axis_length/2} ${wheel_z_offset}" rotate_visual="1" friction="1.0" />
+  <xacro:wheel name="left_rear" xyz="${-wheel_x_offset} ${axis_length/2} ${wheel_z_offset}" rotate_visual="1" friction="1.0" />
+  <xacro:wheel name="right_front" xyz="${wheel_x_offset} ${-axis_length/2} ${wheel_z_offset}" rotate_visual="0" friction="1.0" />
+  <xacro:wheel name="right_rear" xyz="${-wheel_x_offset} ${-axis_length/2} ${wheel_z_offset}" rotate_visual="0" friction="1.0" />
   <link name="base_footprint"/>
   <joint name="base_footprint_joint" type="fixed">
-    <origin xyz="0 0 ${wheel_radius -  wheel_z_offset}" rpy="0 0 0" />
-    <parent link="base_footprint"/>
-    <child link="base_link" />
+    <origin xyz="0 0 ${-(wheel_radius -  wheel_z_offset)}" rpy="0 0 0" />
+    <child link="base_footprint"/>
+    <parent link="base_link" />
   </joint>
   <link name="base_top" />
@@ -92,3 +108,24 @@
     <child link="base_top"/>
   </joint>
+  <gazebo>
+    <plugin name="skid_steer_drive_controller" filename="libgazebo_ros_skid_steer_drive.so">
+      <updateRate>200.0</updateRate>
+      <robotNamespace>/</robotNamespace>
+      <leftFrontJoint>left_front_wheel_joint</leftFrontJoint>
+      <rightFrontJoint>right_front_wheel_joint</rightFrontJoint>
+      <leftRearJoint>left_rear_wheel_joint</leftRearJoint>
+      <rightRearJoint>right_rear_wheel_joint</rightRearJoint>
+      <wheelSeparation>${axis_length}</wheelSeparation>
+      <wheelDiameter>${2*wheel_radius}</wheelDiameter>
+      <robotBaseFrame>base_link</robotBaseFrame>
+      <torque>1</torque>
+      <commandTopic>cmd_vel</commandTopic>
+      <odometryTopic>odom_combined</odometryTopic>
+      <odometryFrame>odom_combined</odometryFrame>
+      <covariance_x>0</covariance_x>
+      <covariance_y>0</covariance_y>
+      <covariance_yaw>0</covariance_yaw>
+      <broadcastTF>True</broadcastTF>
+    </plugin>
+  </gazebo>
 </robot>

Commit message: edited urdf

File: urdf/simplebot.urdf.xacro (robot description, xacro)
@@ -98,7 +98,7 @@
   <link name="base_footprint"/>
   <joint name="base_footprint_joint" type="fixed">
-    <origin xyz="0 0 ${-(wheel_radius -  wheel_z_offset)}" rpy="0 0 0" />
-    <child link="base_footprint"/>
-    <parent link="base_link" />
+    <origin xyz="0 0 ${wheel_radius -  wheel_z_offset}" rpy="0 0 0" />
+    <parent link="base_footprint"/>
+    <child link="base_link" />
   </joint>
   <link name="base_top" />
@@ -118,5 +118,5 @@
       <wheelSeparation>${axis_length}</wheelSeparation>
       <wheelDiameter>${2*wheel_radius}</wheelDiameter>
-      <robotBaseFrame>base_link</robotBaseFrame>
+      <robotBaseFrame>base_footprint</robotBaseFrame>
       <torque>1</torque>
       <commandTopic>cmd_vel</commandTopic>
